File: v1.23/Lotus58_Glow.kicad_sch (KiCad schematic)
At the start: 133 parts, among them J2 Conn_01x02, P1 OLED, SW1 Kailh hotswap MX socket, SW10 Kailh hotswap MX socket, SW11 Kailh hotswap MX socket, SW12 Kailh hotswap MX socket, SW13 Kailh hotswap MX socket, SW14 Kailh hotswap MX socket, SW15 Kailh hotswap MX socket, SW16 Kailh hotswap MX socket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

Commit message: Added viewable schematic
Parts:
- J1: value (none) -> PJ-320A; footprint (none) -> Common Library:MJ-4PP-9_alim
Other:
- moved on the sheet: C1, C10, C11, C2, C3, C4, C5, C6, C7, C8, C9, D1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
