File: v1.24/_autosave-Lotus58_Glow.kicad_sch (KiCad schematic)
At the start: 136 parts, among them J1 PJ-320A, J2 Conn_01x02, P1 OLED, SW1 Kailh hotswap MX socket, SW10 Kailh hotswap MX socket, SW11 Kailh hotswap MX socket, SW12 Kailh hotswap MX socket, SW13 Kailh hotswap MX socket, SW14 Kailh hotswap MX socket, SW15 Kailh hotswap MX socket, SW16 Kailh hotswap MX socket, SW17 Kailh hotswap MX socket, SW18 Kailh hotswap MX socket, SW19 Kailh hotswap MX socket, SW2 Kailh hotswap MX socket, SW20 Kailh hotswap MX socket, SW21 Kailh hotswap MX socket, SW22 Kailh hotswap MX socket, SW23 Kailh hotswap MX socket, SW24 Kailh hotswap MX socket, SW25 Kailh hotswap MX socket, SW26 Kailh hotswap MX socket, SW27 Kailh hotswap MX socket, SW28 Kailh hotswap MX socket, SW29 Kailh hotswap MX socket, SW3 Kailh hotswap MX socket, SW30 Rotary_Encoder_Switch, SW31 Rotary_Encoder_Switch, SW4 Kailh hotswap MX socket, SW5 Kailh hotswap MX socket, SW6 Kailh hotswap MX socket, SW7 Kailh hotswap MX socket, SW8 Kailh hotswap MX socket, SW9 Kailh hotswap MX socket, U1 ProMicro, U2 SRV05-4

Commit message: Update _autosave-Lotus58_Glow.kicad_sch
Parts:
- removed J1: PJ-320A, Common Library:MJ-4PP-9_alim, symbol Connector:AudioJack4
- added D31: SMF5.0CA, Diode_SMD:D_SOD-123, symbol Keyboard Common:SMF5.0CA
- added FB1, FB2, FB3: FerriteBead_Small, Capacitor_SMD:C_0805_2012Metric_Pad1.18x1.45mm_HandSolder, symbol Device:FerriteBead_Small
- added J1, J3: USB_C_Receptacle_USB2.0, Keyboard Common:HRO_TYPE-C-31-M-12, symbol Connector:USB_C_Receptacle_USB2.0
- added Q1: AO3401A, Package_TO_SOT_SMD:SOT-23, symbol Transistor_FET:AO3401A
Connections:
- net DATA: now also J1.A8 (SBU1), J1.B8 (SBU2), J3.A8 (SBU1), J3.B8 (SBU2)
- net GND: now also D31.1 (A1), FB2.2, FB3.2, J1.A1 (GND), J1.A12 (GND), J1.B1 (GND), J1.B12 (GND), J3.A1 (GND), J3.A12 (GND), J3.B1 (GND), J3.B12 (GND), Q1.1 (G)
- net VCC: now also Q1.2 (S)
- new net: FB2.1, FB3.1, J1.S1 (SHIELD), J3.S1 (SHIELD)
- new net VBUS1: FB1.1, J1.A4 (VBUS), J1.A9 (VBUS), J1.B4 (VBUS), J1.B9 (VBUS), J3.A4 (VBUS), J3.A9 (VBUS), J3.B4 (VBUS), J3.B9 (VBUS)
- new net VBUS2: D31.2 (A2), FB1.2, Q1.3 (D)
- no-connect marks 6 -> 17
Other:
- moved on the sheet: C1, C10, C11, C2, C3, C4, C5, C6, C7, C8, C9, J2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
