File: Lotus 58 C v1.0.0/Lotus58_C.kicad_sch (KiCad schematic)
At the start: 136 parts, among them J1 PJ-320A, J2 Conn_01x02, P1 OLED, SW1 Kailh hotswap MX socket, SW10 Kailh hotswap MX socket, SW11 Kailh hotswap MX socket, SW12 Kailh hotswap MX socket, SW13 Kailh hotswap MX socket, SW14 Kailh hotswap MX socket, SW15 Kailh hotswap MX socket, SW16 Kailh hotswap MX socket, SW17 Kailh hotswap MX socket, SW18 Kailh hotswap MX socket, SW19 Kailh hotswap MX socket, SW2 Kailh hotswap MX socket, SW20 Kailh hotswap MX socket, SW21 Kailh hotswap MX socket, SW22 Kailh hotswap MX socket, SW23 Kailh hotswap MX socket, SW24 Kailh hotswap MX socket, SW25 Kailh hotswap MX socket, SW26 Kailh hotswap MX socket, SW27 Kailh hotswap MX socket, SW28 Kailh hotswap MX socket, SW29 Kailh hotswap MX socket, SW3 Kailh hotswap MX socket, SW30 Rotary_Encoder_Switch, SW31 Rotary_Encoder_Switch, SW4 Kailh hotswap MX socket, SW5 Kailh hotswap MX socket, SW6 Kailh hotswap MX socket, SW7 Kailh hotswap MX socket, SW8 Kailh hotswap MX socket, SW9 Kailh hotswap MX socket, U1 ProMicro, U2 SRV05-4

Commit message: Lotus 58 C v1.0.0
Moved to full SMD and USB-C
Parts:
- removed C3, C5, C7, C9: 100nF, Common Library:RESISTOR_Reversible, symbol Device:C_Small
- removed J1: PJ-320A, Common Library:MJ-4PP-9_alim, symbol Connector:AudioJack4
- added D31: SMF5.0CA, Diode_SMD:D_SOD-123, symbol Keyboard Common:SMF5.0CA
- added FB1, FB2: FerriteBead_Small, Capacitor_SMD:C_0805_2012Metric_Pad1.18x1.45mm_HandSolder, symbol Device:FerriteBead_Small
- added J1, J3: USB_C_Receptacle_USB2.0, Keyboard Common:HRO_TYPE-C-31-M-12, symbol Connector:USB_C_Receptacle_USB2.0
- added Q1: AO3401A, Package_TO_SOT_SMD:SOT-23, symbol Transistor_FET:AO3401A
- C1, C2: footprint Common Library:RESISTOR_Reversible -> Capacitor_SMD:C_0603_1608Metric_Pad1.08x0.95mm_HandSolder
- D1, D10, D11, D12, D13, D14, D15, D16, D17, D18, D19, D2, D20, D21, D22, D23, D24, D25, D26, D27, D28, D29, D3, D30, D4, D5, D6, D7, D8, D9: value 1N4148/1N4148W -> 1N4148W; footprint Keyboard Library:Diode_DO35_SOD123 -> Diode_SMD:D_SOD-123
- R1, R2: footprint Resistor_THT:R_Axial_DIN0207_L6.3mm_D2.5mm_P7.62mm_Horizontal -> Resistor_SMD:R_0603_1608Metric_Pad0.98x0.95mm_HandSolder
Connections:
- net DATA: now also U2.4 (IO3), J1.A8 (SBU1), J1.B8 (SBU2), J3.A8 (SBU1), J3.B8 (SBU2); no longer U2.3 (IO2)
- net GND: now also D31.1 (A1), FB2.2, J1.A1 (GND), J1.A12 (GND), J1.B1 (GND), J1.B12 (GND), J3.A1 (GND), J3.A12 (GND), J3.B1 (GND), J3.B12 (GND), Q1.1 (G)
- net VCC: now also Q1.2 (S)
- new net Shield: FB2.1, J1.S1 (SHIELD), J3.S1 (SHIELD)
- new net VBUS1: FB1.1, J1.A4 (VBUS), J1.A9 (VBUS), J1.B4 (VBUS), J1.B9 (VBUS), J3.A4 (VBUS), J3.A9 (VBUS), J3.B4 (VBUS), J3.B9 (VBUS)
- new net VBUS2: D31.2 (A2), FB1.2, Q1.3 (D)
- no-connect marks 6 -> 17
Other:
- title: Lotus 58 Glow -> Lotus 58 C
- moved on the sheet: C1, C10, C11, C2, C4, C6, C8, J2, JP1, JP10, JP11, JP12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

Commit message: Lotus C
Minor tweaks
SMD capacitors
Parts:
- C10, C11, C4, C6, C8: footprint Common Library:RESISTOR_Reversible -> Capacitor_SMD:C_0603_1608Metric_Pad1.08x0.95mm_HandSolder
Changed lines of the file:
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@@
       (effects (font (size 1.27 1.27)) (justify left))
     )
-    (property "Footprint" "Common Library:RESISTOR_Reversible" (id 2) (at 163.83 189.23 0)
+    (property "Footprint" "Capacitor_SMD:C_0603_1608Metric_Pad1.08x0.95mm_HandSolder" (id 2) (at 163.83 189.23 0)
       (effects (font (size 1.27 1.27)) hide)
     )
@@
       (effects (font (size 1.27 1.27)) (justify left))
     )
-    (property "Footprint" "Common Library:RESISTOR_Reversible" (id 2) (at 152.4 223.52 0)
+    (property "Footprint" "Capacitor_SMD:C_0603_1608Metric_Pad1.08x0.95mm_HandSolder" (id 2) (at 152.4 223.52 0)
       (effects (font (size 1.27 1.27)) hide)
     )
@@
       (effects (font (size 1.27 1.27)) (justify left))
     )
-    (property "Footprint" "Common Library:RESISTOR_Reversible" (id 2) (at 163.83 223.52 0)
+    (property "Footprint" "Capacitor_SMD:C_0603_1608Metric_Pad1.08x0.95mm_HandSolder" (id 2) (at 163.83 223.52 0)
       (effects (font (size 1.27 1.27)) hide)
     )
@@
       (effects (font (size 1.27 1.27)) (justify left))
     )
-    (property "Footprint" "Common Library:RESISTOR_Reversible" (id 2) (at 152.4 259.08 0)
+    (property "Footprint" "Capacitor_SMD:C_0603_1608Metric_Pad1.08x0.95mm_HandSolder" (id 2) (at 152.4 259.08 0)
       (effects (font (size 1.27 1.27)) hide)
     )
@@
       (effects (font (size 1.27 1.27)) (justify left))
     )
-    (property "Footprint" "Common Library:RESISTOR_Reversible" (id 2) (at 163.83 259.08 0)
+    (property "Footprint" "Capacitor_SMD:C_0603_1608Metric_Pad1.08x0.95mm_HandSolder" (id 2) (at 163.83 259.08 0)
       (effects (font (size 1.27 1.27)) hide)
     )
@@
     )
     (path "/00000000-0000-0000-0000-000061ffd61d"
-      (reference "C4") (unit 1) (value "100nF") (footprint "Common Library:RESISTOR_Reversible")
+      (reference "C4") (unit 1) (value "100nF") (footprint "Capacitor_SMD:C_0603_1608Metric_Pad1.08x0.95mm_HandSolder")
     )
     (path "/00000000-0000-0000-0000-00006207a238"
-      (reference "C6") (unit 1) (value "100nF") (footprint "Common Library:RESISTOR_Reversible")
+      (reference "C6") (unit 1) (value "100nF") (footprint "Capacitor_SMD:C_0603_1608Metric_Pad1.08x0.95mm_HandSolder")
     )
     (path "/00000000-0000-0000-0000-00006207a244"
-      (reference "C8") (unit 1) (value "100nF") (footprint "Common Library:RESISTOR_Reversible")
+      (reference "C8") (unit 1) (value "100nF") (footprint "Capacitor_SMD:C_0603_1608Metric_Pad1.08x0.95mm_HandSolder")
     )
     (path "/00000000-0000-0000-0000-00006209914b"
-      (reference "C10") (unit 1) (value "100nF") (footprint "Common Library:RESISTOR_Reversible")
+      (reference "C10") (unit 1) (value "100nF") (footprint "Capacitor_SMD:C_0603_1608Metric_Pad1.08x0.95mm_HandSolder")
     )
     (path "/00000000-0000-0000-0000-000062099151"
-      (reference "C11") (unit 1) (value "100nF") (footprint "Common Library:RESISTOR_Reversible")
+      (reference "C11") (unit 1) (value "100nF") (footprint "Capacitor_SMD:C_0603_1608Metric_Pad1.08x0.95mm_HandSolder")
     )
     (path "/00000000-0000-0000-0000-00005b7226e7"
