File: Lotus 58 Glow/v1.24/_autosave-Lotus58_Glow.kicad_pcb (KiCad board)
At the start: 2 copper layers, 139.1 x 107.7 mm, 136 parts, among them J1 PJ-320A, J2 Conn_01x02, P1 OLED, SW1 Kailh hotswap MX socket, SW10 Kailh hotswap MX socket, SW11 Kailh hotswap MX socket, SW12 Kailh hotswap MX socket, SW13 Kailh hotswap MX socket, SW14 Kailh hotswap MX socket, SW15 Kailh hotswap MX socket, SW16 Kailh hotswap MX socket, SW17 Kailh hotswap MX socket, SW18 Kailh hotswap MX socket, SW19 Kailh hotswap MX socket, SW2 Kailh hotswap MX socket, SW20 Kailh hotswap MX socket, SW21 Kailh hotswap MX socket, SW22 Kailh hotswap MX socket, SW23 Kailh hotswap MX socket, SW24 Kailh hotswap MX socket, SW25 Kailh hotswap MX socket, SW26 Kailh hotswap MX socket, SW27 Kailh hotswap MX socket, SW28 Kailh hotswap MX socket, SW29 Kailh hotswap MX socket, SW3 Kailh hotswap MX socket, SW30 Rotary_Encoder_Switch, SW31 Rotary_Encoder_Switch, SW4 Kailh hotswap MX socket, SW5 Kailh hotswap MX socket, SW6 Kailh hotswap MX socket, SW7 Kailh hotswap MX socket, SW8 Kailh hotswap MX socket, SW9 Kailh hotswap MX socket, U1 ProMicro, U2 SRV05-4

Commit message: retrieved old
Parts:
- moved JP3 16.0 mm to (99.8, 71.8)
- moved JP4 16.0 mm to (99.8, 71.8)
- moved R1 3.00 mm to (99.7, 82.5)
- moved R2 3.00 mm to (102.4, 82.5)
- moved JP1 0.46 mm to (83.4, 37.4), turned to 180 degrees
- moved JP2 0.46 mm to (83.4, 37.4), turned to 180 degrees
- moved U2 0.15 mm to (84.2, 75.0), turned to -90 degrees
Connections:
- U2 pad 3: DATA -> unconnected-(U2-Pad3)
- U2 pad 4: unconnected-(U2-Pad4) -> DATA
Routing:
- net VCC: track 880.7 -> 900.9 mm, vias 37 -> 38
- net GND: track 197.5 -> 179.2 mm
- net SDA: track 57.0 -> 62.6 mm
- net SCL: track 65.0 -> 69.7 mm
- net row4: track 158.7 -> 155.9 mm
- net col1: track 247.5 -> 245.7 mm
- net col4: track 184.1 -> 182.5 mm
- net RESET: track 27.2 -> 25.8 mm
- net RGB_LINK: track 104.5 -> 103.4 mm
- net Net-(LED31-Pad1): track 71.9 -> 70.7 mm
- net LED: track 72.7 -> 73.8 mm
- net Net-(LED32-Pad1): track 66.0 -> 64.9 mm
- net Net-(D26-Pad2): track 10.5 -> 9.41 mm
- net Net-(LED22-Pad4): track 21.7 -> 20.7 mm
- net RGB_KEY: track 52.9 -> 53.6 mm
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Other:
- board text added: "Close jumpers for OLED on Left Hand"
- board text added: "Close jumpers for OLED on Right Hand"
- board text added: "Licensed under CERN-OHL-S v2+"
- board text added: "Markus Knutsson 2022 https://github.com/TweetyDaBird"
- board text removed: "Close jumpers for OLED on LEFT HAND"
- board text removed: "Close jumpers for OLED on RIGHT HAND"
- board text removed: "Markus Knutsson 2022 - https://github.com/TweetyDaBird - Licensed under CERN-OHL-S v2+"
- board text removed: "OFF - ON"
