File: Lotus 58 Glow/v1.24/_autosave-Lotus58_Glow.kicad_sch (KiCad schematic)
At the start: 136 parts, among them J1 PJ-320A, J2 Conn_01x02, P1 OLED, SW1 Kailh hotswap MX socket, SW10 Kailh hotswap MX socket, SW11 Kailh hotswap MX socket, SW12 Kailh hotswap MX socket, SW13 Kailh hotswap MX socket, SW14 Kailh hotswap MX socket, SW15 Kailh hotswap MX socket, SW16 Kailh hotswap MX socket, SW17 Kailh hotswap MX socket, SW18 Kailh hotswap MX socket, SW19 Kailh hotswap MX socket, SW2 Kailh hotswap MX socket, SW20 Kailh hotswap MX socket, SW21 Kailh hotswap MX socket, SW22 Kailh hotswap MX socket, SW23 Kailh hotswap MX socket, SW24 Kailh hotswap MX socket, SW25 Kailh hotswap MX socket, SW26 Kailh hotswap MX socket, SW27 Kailh hotswap MX socket, SW28 Kailh hotswap MX socket, SW29 Kailh hotswap MX socket, SW3 Kailh hotswap MX socket, SW30 Rotary_Encoder_Switch, SW31 Rotary_Encoder_Switch, SW4 Kailh hotswap MX socket, SW5 Kailh hotswap MX socket, SW6 Kailh hotswap MX socket, SW7 Kailh hotswap MX socket, SW8 Kailh hotswap MX socket, SW9 Kailh hotswap MX socket, U1 ProMicro, U2 SRV05-4

Commit message: retrieved old
Connections:
- net DATA: now also U2.4 (IO3); no longer U2.3 (IO2)
Changed lines of the file:
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@@
   (no_connect (at 262.89 92.71))
   (no_connect (at 288.29 97.79))
-  (no_connect (at 288.29 92.71))
+  (no_connect (at 262.89 97.79))
   (no_connect (at 318.77 151.13))
   (wire (pts (xy 107.95 156.21) (xy 130.81 156.21))
@@
     )
   )
-  (global_label "DATA" (shape input) (at 262.89 97.79 180) (fields_autoplaced)
-    (effects (font (size 1.27 1.27)) (justify right))
-    (property "Intersheet References" "${INTERSHEET_REFS}" (id 0) (at 607.06 229.87 0)
-      (effects (font (size 1.27 1.27)) hide)
-    )
+  (global_label "DATA" (shape input) (at 288.29 92.71 0) (fields_autoplaced)
+    (effects (font (size 1.27 1.27)) (justify left))
+    (property "Intersheet References" "${INTERSHEET_REFS}" (id 0) (at -55.88 -39.37 0)
+      (effects (font (size 1.27 1.27)) hide)
+    )
