File: Lotus 58 Glow/v1.24/Lotus58_Glow_124.kicad_sch (KiCad schematic)
At the start: 137 parts, among them J1 USB_C_Receptacle_USB2.0, J2 Conn_01x02, J3 USB_C_Receptacle_USB2.0, P1 OLED, Q1 AO3401A, SW1 Kailh hotswap MX socket, SW10 Kailh hotswap MX socket, SW11 Kailh hotswap MX socket, SW12 Kailh hotswap MX socket, SW13 Kailh hotswap MX socket, SW14 Kailh hotswap MX socket, SW15 Kailh hotswap MX socket, SW16 Kailh hotswap MX socket, SW17 Kailh hotswap MX socket, SW18 Kailh hotswap MX socket, SW19 Kailh hotswap MX socket, SW2 Kailh hotswap MX socket, SW20 Kailh hotswap MX socket, SW21 Kailh hotswap MX socket, SW22 Kailh hotswap MX socket, SW23 Kailh hotswap MX socket, SW24 Kailh hotswap MX socket, SW25 Kailh hotswap MX socket, SW26 Kailh hotswap MX socket, SW27 Kailh hotswap MX socket, SW28 Kailh hotswap MX socket, SW29 Kailh hotswap MX socket, SW3 Kailh hotswap MX socket, SW30 Rotary_Encoder_Switch, SW31 Rotary_Encoder_Switch, SW4 Kailh hotswap MX socket, SW5 Kailh hotswap MX socket, SW6 Kailh hotswap MX socket, SW7 Kailh hotswap MX socket, SW8 Kailh hotswap MX socket, SW9 Kailh hotswap MX socket, U1 ProMicro, U2 SRV05-4

Commit message: General cleanup and rename
Parts:
- removed D31: SMF5.0CA, Diode_SMD:D_SOD-123, symbol Keyboard Common:SMF5.0CA
- removed FB1, FB2: FerriteBead_Small, Capacitor_SMD:C_0805_2012Metric_Pad1.18x1.45mm_HandSolder, symbol Device:FerriteBead_Small
- removed J1, J3: USB_C_Receptacle_USB2.0, Keyboard Common:HRO_TYPE-C-31-M-12, symbol Connector:USB_C_Receptacle_USB2.0
- removed Q1: AO3401A, Package_TO_SOT_SMD:SOT-23, symbol Transistor_FET:AO3401A
- added J1: PJ-320A, Common Library:MJ-4PP-9_alim, symbol Connector:AudioJack4
- C1, C2, C4: footprint Capacitor_SMD:C_0603_1608Metric_Pad1.08x0.95mm_HandSolder -> Common Library:RESISTOR_Reversible
- C3: renamed from C11; footprint Capacitor_SMD:C_0603_1608Metric_Pad1.08x0.95mm_HandSolder -> Common Library:RESISTOR_Reversible
- C5: renamed from C6; footprint Capacitor_SMD:C_0603_1608Metric_Pad1.08x0.95mm_HandSolder -> Common Library:RESISTOR_Reversible
- C6: renamed from C8; footprint Capacitor_SMD:C_0603_1608Metric_Pad1.08x0.95mm_HandSolder -> Common Library:RESISTOR_Reversible
- C8: renamed from C10; footprint Capacitor_SMD:C_0603_1608Metric_Pad1.08x0.95mm_HandSolder -> Common Library:RESISTOR_Reversible
- D1, D10, D11, D12, D13, D14, D15, D16, D17, D18, D19, D2, D20, D21, D22, D23, D24, D25, D26, D27, D28, D29, D3, D30, D4, D5, D6, D7, D8, D9: value 1N4148W -> 1N4148/1N4148W; footprint Diode_SMD:D_SOD-123 -> Keyboard Library:Diode_DO35_SOD123
- LED1, LED10, LED11, LED12, LED13, LED14, LED15, LED16, LED17, LED18, LED19, LED2, LED20, LED21, LED22, LED23, LED24, LED25, LED26, LED27, LED28, LED29, LED3, LED4, LED5, LED6, LED7, LED8, LED9: footprint kicad-keyboard-parts:MX_SK6812MINI-E_REVERSIBLE -> Keyboard RGB:MX_SK6812MINI-E_REVERSIBLE
- R1, R2: footprint Resistor_SMD:R_0603_1608Metric_Pad0.98x0.95mm_HandSolder -> Resistor_THT:R_Axial_DIN0207_L6.3mm_D2.5mm_P7.62mm_Horizontal
- S1: footprint MSK12C02 -> Keyboard Common:MSK12C02
- TH1, TH2, TH3, TH4, TH5: footprint MountingHole:MountingHole_3.7mm -> Keyboard Common:Spacer PCB hole
- U1: footprint Keyboard Controllers:ArduinoProMicro-BackSide -> Keyboard Controllers:ProMicro_Reversible_orig
Connections:
- net DATA: now also U2.3 (IO2), J1.R2; no longer U2.4 (IO3)
- net GND: now also J1.R1
- net VCC: now also J1.T
- no-connect marks 17 -> 6
Other:
- title: Lotus 58 C -> Lotus 58 Glow
- moved on the sheet: C1, C2, C3, C4, C5, C6, C8, J2, JP1, JP10, JP11, JP12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

Commit message: v1.2.4
Ordered prototype
Parts:
- removed R1, R2: 4k7, Resistor_THT:R_Axial_DIN0207_L6.3mm_D2.5mm_P7.62mm_Horizontal, symbol Device:R
- added Logo1: QMK_Logo, Logotypes:qmk logo, symbol Logotypes:QMK_Logo
- renumbered C4 to C3, C5 to C4, C6 to C5, C8 to C6, C3 to C7, JP6 to JP10, JP7 to JP11, JP8 to JP12, JP9 to JP13, JP10 to JP14, JP11 to JP15, JP12 to JP16, JP3 to JP2, JP4 to JP3, JP2 to JP4, JP13 to JP5, JP14 to JP6, JP16 to JP7, JP15 to JP8, JP5 to JP9, LED30 to LED1, LED4 to LED10, LED5 to LED11, LED6 to LED12, LED7 to LED13, LED8 to LED14, LED9 to LED15, LED10 to LED16, LED11 to LED17, LED12 to LED18, LED13 to LED19, LED31 to LED2, LED14 to LED20, LED15 to LED21, LED16 to LED22, LED17 to LED23, LED18 to LED24, LED19 to LED25, LED20 to LED26, LED21 to LED27, LED22 to LED28, LED23 to LED29, LED32 to LED3, LED24 to LED30, LED25 to LED31, LED26 to LED32, LED27 to LED33, LED28 to LED34, LED29 to LED35, LED33 to LED4, LED34 to LED5, LED35 to LED6, LED1 to LED7, LED2 to LED8, LED3 to LED9
