File: Lotus 58 Glow/v1.24/Lotus58_Glow-backups/Lotus58_Glow-2022-03-10_084902/Lotus58_Glow.kicad_pcb (KiCad board)
At the start: 2 copper layers, 139.1 x 107.7 mm, 136 parts, among them J1 PJ-320A, J2 Conn_01x02, P1 OLED, SW1 Kailh hotswap MX socket, SW10 Kailh hotswap MX socket, SW11 Kailh hotswap MX socket, SW12 Kailh hotswap MX socket, SW13 Kailh hotswap MX socket, SW14 Kailh hotswap MX socket, SW15 Kailh hotswap MX socket, SW16 Kailh hotswap MX socket, SW17 Kailh hotswap MX socket, SW18 Kailh hotswap MX socket, SW19 Kailh hotswap MX socket, SW2 Kailh hotswap MX socket, SW20 Kailh hotswap MX socket, SW21 Kailh hotswap MX socket, SW22 Kailh hotswap MX socket, SW23 Kailh hotswap MX socket, SW24 Kailh hotswap MX socket, SW25 Kailh hotswap MX socket, SW26 Kailh hotswap MX socket, SW27 Kailh hotswap MX socket, SW28 Kailh hotswap MX socket, SW29 Kailh hotswap MX socket, SW3 Kailh hotswap MX socket, SW30 Rotary_Encoder_Switch, SW31 Rotary_Encoder_Switch, SW4 Kailh hotswap MX socket, SW5 Kailh hotswap MX socket, SW6 Kailh hotswap MX socket, SW7 Kailh hotswap MX socket, SW8 Kailh hotswap MX socket, SW9 Kailh hotswap MX socket, U1 ProMicro, U2 SRV05-4

Commit message: retrieved old
Parts:
- removed JP13, JP14: FULL, Common Library:Jumper_Mini
- removed U2: SRV05-4, Package_TO_SOT_SMD:SOT-23-6
- C1, C10, C11, C2, C3, C4, C5, C6, C7, C8, C9: footprint Common Library:RESISTOR_Reversible -> Keyboard Library:RESISTOR_Reversible
- JP1, JP10, JP11, JP12, JP15, JP2, JP3, JP4, JP5, JP6, JP7, JP8, JP9: footprint Common Library:Jumper_Mini -> Keyboard Library:Jumper_Mini
- JP16: value FULL -> RGB; footprint Common Library:Jumper_Mini -> Jumper:SolderJumper-3_P1.3mm_Open_Pad1.0x1.5mm
- S1: footprint Keyboard Common:MSK12C02 -> Keyboard Switches & Encoders:MSK12C02
- moved JP15 7.96 mm to (101.7, 98.3), turned to 180 degrees
- moved JP16 1.40 mm to (101.9, 89.7), turned to 90 degrees
- moved JP3 1.00 mm to (83.8, 72.9), turned to -90 degrees
- moved JP4 1.00 mm to (83.8, 72.9), turned to -90 degrees
- moved D30 0.42 mm to (91.7, 77.7)
Connections:
- JP16 pad 1: LED -> RGB_KEY
- JP16 pad 2: RGB_KEY -> LED
Routing:
- net GND: track 197.5 -> 187.4 mm, vias 97 -> 92
- net RGB_LINK: track 104.5 -> 97.9 mm
- net VCC: track 880.7 -> 886.8 mm
- net DATA: track 66.1 -> 62.1 mm, vias 1 -> 0
- net LED: track 72.7 -> 69.0 mm
- net RGB_KEY: track 52.9 -> 50.8 mm, vias 4 -> 3
- net RGB_GLOW: track 28.8 -> 27.4 mm
- net Hand: track 22.9 -> 22.2 mm
- net row4: track 158.7 -> 159.4 mm
Other:
- board text added: "Capactitors C3 to C11 are optional, and can be left unused."
- board text added: "D30 is optional, and only needed if the encoder is placed in the top position."
- board text added: "Do NOT solder TRRS if building a wireless keyboard"
- board text added: "Encoder Capacitors"
- board text added: "Markus Knutsson 2021 - https://github.com/TweetyDaBird - Licensed under CERN-OHL-S v2+"
- board text added: "OLED Resistors"
- board text added: "Place ProMicro or socket in markings with component side against PCB"
- board text added: "Warning: Close ONLY one RGB connection!"
- board text added: "v1.23"
- board text removed: "Capactitors C3 to C11 are only used if battery operated"
- board text removed: "FULL RGB"
- board text removed: "Left Hand: Encoder Capacitors"
- board text removed: "Left Hand: OLED Resistors"
- board text removed: "Left Hand: Place ProMicro or socket in markings with component side against PCB"
- board text removed: "Markus Knutsson 2022 - https://github.com/TweetyDaBird - Licensed under CERN-OHL-S v2+"
- board text removed: "RESET"
- board text removed: "RGB SETUP"
- board text removed: "Right Hand: Encoder Capacitors"
- board text removed: "Right Hand: OLED Resistors"
- board text removed: "Right Hand: Place ProMicro or socket in markings with component side against PCB"
- board text removed: "TRRS NOT soldered for wireless"
- board text removed: "v1.24"
