File: Lotus 58 Glow/v1.24/Lotus58_Glow-backups/Lotus58_Glow-2022-03-10_084902/Lotus58_Glow.kicad_sch (KiCad schematic)
At the start: 136 parts, among them J1 PJ-320A, J2 Conn_01x02, P1 OLED, SW1 Kailh hotswap MX socket, SW10 Kailh hotswap MX socket, SW11 Kailh hotswap MX socket, SW12 Kailh hotswap MX socket, SW13 Kailh hotswap MX socket, SW14 Kailh hotswap MX socket, SW15 Kailh hotswap MX socket, SW16 Kailh hotswap MX socket, SW17 Kailh hotswap MX socket, SW18 Kailh hotswap MX socket, SW19 Kailh hotswap MX socket, SW2 Kailh hotswap MX socket, SW20 Kailh hotswap MX socket, SW21 Kailh hotswap MX socket, SW22 Kailh hotswap MX socket, SW23 Kailh hotswap MX socket, SW24 Kailh hotswap MX socket, SW25 Kailh hotswap MX socket, SW26 Kailh hotswap MX socket, SW27 Kailh hotswap MX socket, SW28 Kailh hotswap MX socket, SW29 Kailh hotswap MX socket, SW3 Kailh hotswap MX socket, SW30 Rotary_Encoder_Switch, SW31 Rotary_Encoder_Switch, SW4 Kailh hotswap MX socket, SW5 Kailh hotswap MX socket, SW6 Kailh hotswap MX socket, SW7 Kailh hotswap MX socket, SW8 Kailh hotswap MX socket, SW9 Kailh hotswap MX socket, U1 ProMicro, U2 SRV05-4

Commit message: retrieved old
Parts:
- removed JP13, JP14, JP16: FULL, Common Library:Jumper_Mini, symbol Device:Jumper_NO_Small
- removed U2: SRV05-4, Package_TO_SOT_SMD:SOT-23-6, symbol Power_Protection:SRV05-4
- added JP16: RGB, Jumper:SolderJumper-3_P1.3mm_Open_Pad1.0x1.5mm, symbol Jumper:Jumper_3_Open
- C1, C10, C11, C2, C3, C4, C5, C6, C7, C8, C9: footprint Common Library:RESISTOR_Reversible -> Keyboard Library:RESISTOR_Reversible
- J1: value PJ-320A -> (none); footprint Common Library:MJ-4PP-9_alim -> (none)
- JP1, JP10, JP11, JP12, JP15, JP2, JP3, JP4, JP5, JP6, JP7, JP8, JP9: footprint Common Library:Jumper_Mini -> Keyboard Library:Jumper_Mini
Connections:
- net LED: now also JP16.2 (C)
- net RGB_GLOW: now also JP16.3 (B)
- net RGB_KEY: now also JP16.1 (A)
- no-connect marks 6 -> 3
Other:
- moved on the sheet: C1, C10, C11, C2, C3, C4, C5, C6, C7, C8, C9, D1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
