File: Lotus 58 Glow/v1.25/Lotus58_Glow-backups/Lotus58_Glow-2022-03-10_084902/Lotus58_Glow.kicad_sch (KiCad schematic)
At the start: 137 parts, among them J1 USB_C_Receptacle_USB2.0, J2 Conn_01x02, J3 USB_C_Receptacle_USB2.0, P1 OLED, Q1 AO3401A, SW1 Kailh hotswap MX socket, SW10 Kailh hotswap MX socket, SW11 Kailh hotswap MX socket, SW12 Kailh hotswap MX socket, SW13 Kailh hotswap MX socket, SW14 Kailh hotswap MX socket, SW15 Kailh hotswap MX socket, SW16 Kailh hotswap MX socket, SW17 Kailh hotswap MX socket, SW18 Kailh hotswap MX socket, SW19 Kailh hotswap MX socket, SW2 Kailh hotswap MX socket, SW20 Kailh hotswap MX socket, SW21 Kailh hotswap MX socket, SW22 Kailh hotswap MX socket, SW23 Kailh hotswap MX socket, SW24 Kailh hotswap MX socket, SW25 Kailh hotswap MX socket, SW26 Kailh hotswap MX socket, SW27 Kailh hotswap MX socket, SW28 Kailh hotswap MX socket, SW29 Kailh hotswap MX socket, SW3 Kailh hotswap MX socket, SW30 Rotary_Encoder_Switch, SW31 Rotary_Encoder_Switch, SW4 Kailh hotswap MX socket, SW5 Kailh hotswap MX socket, SW6 Kailh hotswap MX socket, SW7 Kailh hotswap MX socket, SW8 Kailh hotswap MX socket, SW9 Kailh hotswap MX socket, U1 ProMicro, U2 SRV05-4

Commit message: General cleanup and rename
Parts:
- removed D31: SMF5.0CA, Diode_SMD:D_SOD-123, symbol Keyboard Common:SMF5.0CA
- removed FB1, FB2: FerriteBead_Small, Capacitor_SMD:C_0805_2012Metric_Pad1.18x1.45mm_HandSolder, symbol Device:FerriteBead_Small
- removed J1, J3: USB_C_Receptacle_USB2.0, Keyboard Common:HRO_TYPE-C-31-M-12, symbol Connector:USB_C_Receptacle_USB2.0
- removed JP13, JP14, JP16: FULL, Common Library:Jumper_Mini, symbol Device:Jumper_NO_Small
- removed Q1: AO3401A, Package_TO_SOT_SMD:SOT-23, symbol Transistor_FET:AO3401A
- removed U2: SRV05-4, Package_TO_SOT_SMD:SOT-23-6, symbol Power_Protection:SRV05-4
- added C3, C5, C7, C9: 100nF, Keyboard Library:RESISTOR_Reversible, symbol Device:C_Small
- added J1: (no value), symbol Connector:AudioJack4
- added JP16: RGB, Jumper:SolderJumper-3_P1.3mm_Open_Pad1.0x1.5mm, symbol Jumper:Jumper_3_Open
- C1, C10, C11, C2, C4, C6, C8: footprint Capacitor_SMD:C_0603_1608Metric_Pad1.08x0.95mm_HandSolder -> Keyboard Library:RESISTOR_Reversible
- D1, D10, D11, D12, D13, D14, D15, D16, D17, D18, D19, D2, D20, D21, D22, D23, D24, D25, D26, D27, D28, D29, D3, D30, D4, D5, D6, D7, D8, D9: value 1N4148W -> 1N4148/1N4148W; footprint Diode_SMD:D_SOD-123 -> Keyboard Library:Diode_DO35_SOD123
- JP1, JP10, JP11, JP12, JP15, JP2, JP3, JP4, JP5, JP6, JP7, JP8, JP9: footprint Common Library:Jumper_Mini -> Keyboard Library:Jumper_Mini
- R1, R2: footprint Resistor_SMD:R_0603_1608Metric_Pad0.98x0.95mm_HandSolder -> Resistor_THT:R_Axial_DIN0207_L6.3mm_D2.5mm_P7.62mm_Horizontal
- U1: footprint Keyboard Controllers:ArduinoProMicro-BackSide -> Keyboard Library:ProMicro_Reversible
Connections:
- net DATA: now also J1.R2
- net GND: now also C3.2, C5.2, C7.2, C9.2, J1.R1
- net LED: now also JP16.2 (C)
- net RGB_GLOW: now also JP16.3 (B)
- net RGB_KEY: now also JP16.1 (A)
- net VCC: now also C3.1, C5.1, C7.1, C9.1, J1.T
- no-connect marks 17 -> 3
Other:
- title: Lotus 58 C -> Lotus 58 Glow
- moved on the sheet: C1, C10, C11, C2, C4, C6, C8, D1, D10, D11, D12, D13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
