File: Lotus 58 WL/v1.0.0/Lotus58_Glow_124.kicad_pcb (KiCad board)
At the start: 2 copper layers, 139.1 x 107.7 mm, 132 parts, among them J1 PJ-320A, J2 Conn_01x02, P1 OLED, SW1 Kailh hotswap MX socket, SW10 Kailh hotswap MX socket, SW11 Kailh hotswap MX socket, SW12 Kailh hotswap MX socket, SW13 Kailh hotswap MX socket, SW14 Kailh hotswap MX socket, SW15 Kailh hotswap MX socket, SW16 Kailh hotswap MX socket, SW17 Kailh hotswap MX socket, SW18 Kailh hotswap MX socket, SW19 Kailh hotswap MX socket, SW2 Kailh hotswap MX socket, SW20 Kailh hotswap MX socket, SW21 Kailh hotswap MX socket, SW22 Kailh hotswap MX socket, SW23 Kailh hotswap MX socket, SW24 Kailh hotswap MX socket, SW25 Kailh hotswap MX socket, SW26 Kailh hotswap MX socket, SW27 Kailh hotswap MX socket, SW28 Kailh hotswap MX socket, SW29 Kailh hotswap MX socket, SW3 Kailh hotswap MX socket, SW30 Rotary_Encoder_Switch, SW31 Rotary_Encoder_Switch, SW4 Kailh hotswap MX socket, SW5 Kailh hotswap MX socket, SW6 Kailh hotswap MX socket, SW7 Kailh hotswap MX socket, SW8 Kailh hotswap MX socket, SW9 Kailh hotswap MX socket, U1 ProMicro, U2 SRV05-4

Commit message: created wireless
Parts:
- removed R1, R2: 4k7, Resistor_THT:R_Axial_DIN0207_L6.3mm_D2.5mm_P7.62mm_Horizontal
- added Logo1: QMK_Logo, Logotypes:qmk logo, B.Cu at (152.9, 112.0)
- U1: footprint Keyboard Library:ProMicro_Reversible -> Keyboard Controllers:ProMicro_Reversible_orig
- moved JP2 3.29 mm to (99.8, 75.1), turned to -90 degrees
- moved JP3 3.29 mm to (99.8, 75.1), turned to -90 degrees
- moved U1 1.20 mm to (92.1, 56.1)
- moved JP1 0.64 mm to (83.3, 38.1)
- moved JP4 0.64 mm to (83.3, 38.1)
- renumbered C4 to C3, C5 to C4, C6 to C5, C8 to C6, C3 to C7, JP6 to JP10, JP7 to JP11, JP8 to JP12, JP9 to JP13, JP10 to JP14, JP11 to JP15, JP12 to JP16, JP3 to JP2, JP4 to JP3, JP2 to JP4, JP13 to JP5, JP14 to JP6, JP16 to JP7, JP15 to JP8, JP5 to JP9, LED30 to LED1, LED4 to LED10, LED5 to LED11, LED6 to LED12, LED7 to LED13, LED8 to LED14, LED9 to LED15, LED10 to LED16, LED11 to LED17, LED12 to LED18, LED13 to LED19, LED31 to LED2, LED14 to LED20, LED15 to LED21, LED16 to LED22, LED17 to LED23, LED18 to LED24, LED19 to LED25, LED20 to LED26, LED21 to LED27, LED22 to LED28, LED23 to LED29, LED32 to LED3, LED24 to LED30, LED25 to LED31, LED26 to LED32, LED27 to LED33, LED28 to LED34, LED29 to LED35, LED33 to LED4, LED34 to LED5, LED35 to LED6, LED1 to LED7, LED2 to LED8, LED3 to LED9
Routing:
- net SCL: track 69.7 -> 47.8 mm
- net GND: track 180.0 -> 197.1 mm, vias 97 -> 90
- net SDA: track 62.7 -> 52.7 mm, vias 2 -> 3
- net VCC: track 905.0 -> 900.8 mm
- net col1: track 246.4 -> 243.6 mm
- net LED: track 73.8 -> 71.5 mm
- net A: track 83.9 -> 85.9 mm, vias 1 -> 0
- net RGB_KEY: track 53.6 -> 51.8 mm
- net col0: track 215.9 -> 214.1 mm
- net row3: track 172.1 -> 170.3 mm
- net row4: track 155.9 -> 154.8 mm
- net Hand: track 22.6 -> 21.8 mm, vias 0 -> 1
- net row2: track 157.7 -> 156.9 mm
- net col5: track 141.2 -> 140.4 mm
- net row0: track 166.9 -> 166.2 mm
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Other:
- board text added: "1. Pick hand/side and close jumpers (hand/OLED/RGB) as labeled for that hand."
- board text added: "2. Solder ALL basic components to the component side (backside) (diodes/hot-swap sockets/capacitors/TRRS). Save the diode legs for later!"
- board text added: "3. Place and solder the RGB LEDS from the component side (key/glow) as marked. 4. Solder controller/sockets in place as marked on the component side. (Use diode legs!)"
- board text added: "5. Solder OLED/Encoder on FRONT of PCB. 6. ESD protection and battery/switch fits one place only."
- board text added: "Capactitors C3 to C8 are optional and only needed if battery operated (or RGB unstable)"
- board text added: "ESD"
- board text added: "Even if you do not socket the controller as recommended, Pretty please! Do NOT use pins supplied with ProMicro!"
- board text added: "Markus Knutsson - 2022 - https://github.com/TweetyDaBird Licensed under CERN-OHL-S v2+"
- board text added: "Place ProMicro or socket in markings with component side against PCB"
- board text added: "Resistors and capacitors can be placed in either direction. Diodes must be placed with the stripe on the body at the line/side where arrow is pointing."
- board text added: "TRRS should NOT BE USED for wireless"
- board text added: "Underglow RGB's are placed with the visible marking matching the notch on its face. Per key RGB's are placed face down, with the notched corner at the VISIBLE marking as they are soldered."
- board text added: "WARNING! Full RGB will overpower the USB fuses! Lower the brightness!"
- board text removed: "Capactitors C3 to C8 are only needed if battery operated"
- board text removed: "Diodes and RGB's MUST be placed in the correct direction to function."
- board text removed: "Left Hand: OLED Resistors"
- board text removed: "Left Hand: Place ProMicro or socket in markings with component side against PCB"
- board text removed: "Licensed under CERN-OHL-S v2+"
- board text removed: "Markus Knutsson 2022 https://github.com/TweetyDaBird"
- board text removed: "Per key RGB's are placed face down, with the notched corner at the VISIBLE marking as they are soldered."
- board text removed: "Place stripe of diode at the line/side where arrow is pointing."
- board text removed: "Resistors and capacitors can be placed in either direction."
- board text removed: "Right Hand: OLED Resistors"
- board text removed: "Right Hand: Place ProMicro or socket in markings with component side against PCB"
- board text removed: "TRRS NOT soldered for wireless"
- board text removed: "The COMPONENT side of the PCB is the BACK side for that hand."
- board text removed: "Underglow RGB's are placed with the visible marking matching the notch on its face."
- board text removed: "WARNING! Full RB is NOT recommended for power consumption reasons."
