File: Lotus 58 WL/v1.0.0/Lotus58_Glow_124.kicad_sch (KiCad schematic)
At the start: 132 parts, among them J1 PJ-320A, J2 Conn_01x02, P1 OLED, SW1 Kailh hotswap MX socket, SW10 Kailh hotswap MX socket, SW11 Kailh hotswap MX socket, SW12 Kailh hotswap MX socket, SW13 Kailh hotswap MX socket, SW14 Kailh hotswap MX socket, SW15 Kailh hotswap MX socket, SW16 Kailh hotswap MX socket, SW17 Kailh hotswap MX socket, SW18 Kailh hotswap MX socket, SW19 Kailh hotswap MX socket, SW2 Kailh hotswap MX socket, SW20 Kailh hotswap MX socket, SW21 Kailh hotswap MX socket, SW22 Kailh hotswap MX socket, SW23 Kailh hotswap MX socket, SW24 Kailh hotswap MX socket, SW25 Kailh hotswap MX socket, SW26 Kailh hotswap MX socket, SW27 Kailh hotswap MX socket, SW28 Kailh hotswap MX socket, SW29 Kailh hotswap MX socket, SW3 Kailh hotswap MX socket, SW30 Rotary_Encoder_Switch, SW31 Rotary_Encoder_Switch, SW4 Kailh hotswap MX socket, SW5 Kailh hotswap MX socket, SW6 Kailh hotswap MX socket, SW7 Kailh hotswap MX socket, SW8 Kailh hotswap MX socket, SW9 Kailh hotswap MX socket, U1 ProMicro, U2 SRV05-4

Commit message: created wireless
Parts:
- removed R1, R2: 4k7, Resistor_THT:R_Axial_DIN0207_L6.3mm_D2.5mm_P7.62mm_Horizontal, symbol Device:R
- added Logo1: QMK_Logo, Logotypes:qmk logo, symbol Logotypes:QMK_Logo
- U1: footprint Keyboard Library:ProMicro_Reversible -> Keyboard Controllers:ProMicro_Reversible_orig
- renumbered C4 to C3, C5 to C4, C6 to C5, C8 to C6, C3 to C7, JP6 to JP10, JP7 to JP11, JP8 to JP12, JP9 to JP13, JP10 to JP14, JP11 to JP15, JP12 to JP16, JP3 to JP2, JP4 to JP3, JP2 to JP4, JP13 to JP5, JP14 to JP6, JP16 to JP7, JP15 to JP8, JP5 to JP9, LED30 to LED1, LED4 to LED10, LED5 to LED11, LED6 to LED12, LED7 to LED13, LED8 to LED14, LED9 to LED15, LED10 to LED16, LED11 to LED17, LED12 to LED18, LED13 to LED19, LED31 to LED2, LED14 to LED20, LED15 to LED21, LED16 to LED22, LED17 to LED23, LED18 to LED24, LED19 to LED25, LED20 to LED26, LED21 to LED27, LED22 to LED28, LED23 to LED29, LED32 to LED3, LED24 to LED30, LED25 to LED31, LED26 to LED32, LED27 to LED33, LED28 to LED34, LED29 to LED35, LED33 to LED4, LED34 to LED5, LED35 to LED6, LED1 to LED7, LED2 to LED8, LED3 to LED9
