File: Lotus 58 Classic/v1.26/Lotus58_Glow_126.kicad_pcb (KiCad board)
At the start: 2 copper layers, 139.1 x 107.7 mm, 125 parts, among them J1 PJ-320A, J2 Conn_01x02, P1 OLED, SW1 Kailh hotswap MX socket, SW10 Kailh hotswap MX socket, SW11 Kailh hotswap MX socket, SW12 Kailh hotswap MX socket, SW13 Kailh hotswap MX socket, SW14 Kailh hotswap MX socket, SW15 Kailh hotswap MX socket, SW16 Kailh hotswap MX socket, SW17 Kailh hotswap MX socket, SW18 Kailh hotswap MX socket, SW19 Kailh hotswap MX socket, SW2 Kailh hotswap MX socket, SW20 Kailh hotswap MX socket, SW21 Kailh hotswap MX socket, SW22 Kailh hotswap MX socket, SW23 Kailh hotswap MX socket, SW24 Kailh hotswap MX socket, SW25 Kailh hotswap MX socket, SW26 Kailh hotswap MX socket, SW27 Kailh hotswap MX socket, SW28 Kailh hotswap MX socket, SW29 Kailh hotswap MX socket, SW3 Kailh hotswap MX socket, SW30 Rotary_Encoder_Switch, SW31 Rotary_Encoder_Switch, SW4 Kailh hotswap MX socket, SW5 Kailh hotswap MX socket, SW6 Kailh hotswap MX socket, SW7 Kailh hotswap MX socket, SW8 Kailh hotswap MX socket, SW9 Kailh hotswap MX socket, U1 ProMicro, U2 SRV05-4

Commit message: v1.26 final
Parts:
- removed JP1, JP4: RESET, Common Library:Jumper_Mini
- added RES1: TS-A002, Keyboard Common:YTS-A002, B.Cu at (118.9, 37.2)
- added RES2: TS-A002, Keyboard Common:YTS-A002, F.Cu at (118.9, 37.2)
- added S2: MSK12C02, Keyboard Common:MSK12C02, B.Cu at (108.7, 37.5)
- SW1, SW10, SW11, SW12, SW13, SW14, SW15, SW16, SW17, SW18, SW19, SW2, SW20, SW21, SW22, SW23, SW24, SW25, SW26, SW27, SW28, SW29, SW3, SW4, SW5, SW6, SW7, SW8, SW9: footprint keyswitches:Kailh_socket_MX_reversible_RGB -> Keyboard Switches:SW_MX_HotSwap_Reversible; moved to B.Cu
- moved S1 2.99 mm to (108.7, 37.5)
- moved D1 0.26 mm to (114.5, 41.7)
- turned SW1 to 180 degrees
- turned SW10 to 180 degrees
- turned SW11 to 180 degrees
- turned SW12 to 180 degrees
- turned SW13 to 180 degrees
- turned SW14 to 180 degrees
- turned SW15 to 180 degrees
- turned SW16 to 180 degrees
- turned SW17 to 180 degrees
- turned SW18 to 180 degrees
- turned SW19 to 180 degrees
- turned SW2 to 180 degrees
- turned SW20 to 180 degrees
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Routing:
- net RESET: track 26.4 -> 48.1 mm, vias 2 -> 4
- net col1: track 238.7 -> 257.1 mm
- net Battery: track 20.2 -> 28.9 mm, vias 0 -> 2
- net GND: track 179.8 -> 186.9 mm, vias 89 -> 100
- net /Batt: track 6.11 -> 8.89 mm, vias 0 -> 1
- net col4: track 180.9 -> 183.3 mm
- net col2: track 220.2 -> 221.8 mm
- net col5: track 137.3 -> 136.0 mm
- net col0: track 213.7 -> 214.9 mm
- net Net-(D26-A): track 9.41 -> 10.4 mm
- net Alt: track 16.5 -> 15.8 mm
- net /PWR_KEY: track 695.7 -> 696.3 mm
- net Net-(LED2-DOUT): track 44.7 -> 45.4 mm
- net /PWR_GLOW: track 301.3 -> 302.0 mm
- net Net-(LED23-DOUT): track 20.7 -> 21.3 mm
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Other:
- board text removed: "RESET"
