File: Lotus 58 Classic/v1.26/Lotus58_Glow_126.kicad_sch (KiCad schematic)
At the start: 125 parts, among them J1 PJ-320A, J2 Conn_01x02, P1 OLED, SW1 Kailh hotswap MX socket, SW10 Kailh hotswap MX socket, SW11 Kailh hotswap MX socket, SW12 Kailh hotswap MX socket, SW13 Kailh hotswap MX socket, SW14 Kailh hotswap MX socket, SW15 Kailh hotswap MX socket, SW16 Kailh hotswap MX socket, SW17 Kailh hotswap MX socket, SW18 Kailh hotswap MX socket, SW19 Kailh hotswap MX socket, SW2 Kailh hotswap MX socket, SW20 Kailh hotswap MX socket, SW21 Kailh hotswap MX socket, SW22 Kailh hotswap MX socket, SW23 Kailh hotswap MX socket, SW24 Kailh hotswap MX socket, SW25 Kailh hotswap MX socket, SW26 Kailh hotswap MX socket, SW27 Kailh hotswap MX socket, SW28 Kailh hotswap MX socket, SW29 Kailh hotswap MX socket, SW3 Kailh hotswap MX socket, SW30 Rotary_Encoder_Switch, SW31 Rotary_Encoder_Switch, SW4 Kailh hotswap MX socket, SW5 Kailh hotswap MX socket, SW6 Kailh hotswap MX socket, SW7 Kailh hotswap MX socket, SW8 Kailh hotswap MX socket, SW9 Kailh hotswap MX socket, U1 ProMicro, U2 SRV05-4

Commit message: v1.26 final
Parts:
- removed JP1, JP4: RESET, Common Library:Jumper_Mini, symbol Device:Jumper_NO_Small
- added RES1, RES2: TS-A002, Keyboard Common:YTS-A002, symbol Keyboard Common:TS-A002
- added S2, S3: MSK12C02, Keyboard Common:MSK12C02, symbol Keyboard Common:MSK12C02
- S1: symbol Keyboard_Library:MSK12C02 -> Keyboard Common:MSK12C02
Connections:
- net Batt: now also S1.COM, S2.COM; no longer S1.B1 (COM)
- net Battery: now also S1.NC, S2.NC; no longer S1.C1 (NO)
- net GND: now also RES1.2, RES1.3, RES2.2, RES2.3, S2.MP (GND), S3.MP (GND)
- net PWR_GLOW: now also S3.NO
- net PWR_KEY: now also S3.NC
- net RESET: now also RES1.1, RES2.1
- net VCC: now also S3.COM
- net col5: now also SW1.2; no longer SW1.1
- net at D1.2 (A): now also SW1.1; no longer SW1.2
- new net: S1.NO, S2.NO
