File: Lotus 58 USB-C/v1.33/Lotus58_Glow_133.kicad_pcb (KiCad board)
At the start: 2 copper layers, 139.1 x 107.7 mm, 117 parts, among them J3 USB_C_Receptacle_USB2.0, P1 OLED, SW1 Kailh hotswap MX socket, SW10 Kailh hotswap MX socket, SW11 Kailh hotswap MX socket, SW12 Kailh hotswap MX socket, SW13 Kailh hotswap MX socket, SW14 Kailh hotswap MX socket, SW15 Kailh hotswap MX socket, SW16 Kailh hotswap MX socket, SW17 Kailh hotswap MX socket, SW18 Kailh hotswap MX socket, SW19 Kailh hotswap MX socket, SW2 Kailh hotswap MX socket, SW20 Kailh hotswap MX socket, SW21 Kailh hotswap MX socket, SW22 Kailh hotswap MX socket, SW23 Kailh hotswap MX socket, SW24 Kailh hotswap MX socket, SW25 Kailh hotswap MX socket, SW26 Kailh hotswap MX socket, SW27 Kailh hotswap MX socket, SW28 Kailh hotswap MX socket, SW29 Kailh hotswap MX socket, SW3 Kailh hotswap MX socket, SW30 Rotary_Encoder_Switch, SW31 Rotary_Encoder_Switch, SW32 MSK12C02, SW33 MSK12C02, SW4 Kailh hotswap MX socket, SW5 Kailh hotswap MX socket, SW6 Kailh hotswap MX socket, SW7 Kailh hotswap MX socket, SW8 Kailh hotswap MX socket, SW9 Kailh hotswap MX socket, U1 ProMicro, U2 SRV05-4

Commit message: Corrected filename for v1.33 files
Routing:
- net /PWR_KEY: track 699.2 -> 699.9 mm
- net Net-(LED31-DOUT): track 43.7 -> 44.3 mm
- net /PWR_GLOW: track 307.7 -> 307.1 mm
- net Net-(LED32-DOUT): track 70.7 -> 70.1 mm
- net GND: track 135.4 -> 135.9 mm

Commit message: Fixed silk screen inconsistencies
Connections:
- J3 pad B8: unconnected-(J3-SBU2-PadB8) -> DATA
Routing:
- net DATA: track 61.2 -> 64.1 mm
Other:
- board text added: "v1.3.3"
- board text removed: "v1.3.1"
