File: Lotus 58 Classic/v1.27/Lotus58_Glow_127.kicad_pcb (KiCad board)
At the start: 2 copper layers, 139.1 x 107.7 mm, 127 parts, among them J1 PJ-320A, J2 Conn_01x02, P1 OLED, SW1 Kailh hotswap MX socket, SW10 Kailh hotswap MX socket, SW11 Kailh hotswap MX socket, SW12 Kailh hotswap MX socket, SW13 Kailh hotswap MX socket, SW14 Kailh hotswap MX socket, SW15 Kailh hotswap MX socket, SW16 Kailh hotswap MX socket, SW17 Kailh hotswap MX socket, SW18 Kailh hotswap MX socket, SW19 Kailh hotswap MX socket, SW2 Kailh hotswap MX socket, SW20 Kailh hotswap MX socket, SW21 Kailh hotswap MX socket, SW22 Kailh hotswap MX socket, SW23 Kailh hotswap MX socket, SW24 Kailh hotswap MX socket, SW25 Kailh hotswap MX socket, SW26 Kailh hotswap MX socket, SW27 Kailh hotswap MX socket, SW28 Kailh hotswap MX socket, SW29 Kailh hotswap MX socket, SW3 Kailh hotswap MX socket, SW30 Rotary_Encoder_Switch, SW31 Rotary_Encoder_Switch, SW4 Kailh hotswap MX socket, SW5 Kailh hotswap MX socket, SW6 Kailh hotswap MX socket, SW7 Kailh hotswap MX socket, SW8 Kailh hotswap MX socket, SW9 Kailh hotswap MX socket, U1 ProMicro, U2 SRV05-4

Commit message: Created STEP files for 3D model
Signed-off-by: TweetyDaBird <markus.knutsson@tweety.se>
Parts:
- removed JP10, JP11, JP12, JP13, JP14, JP15, JP16, JP9: Jumper_NO_Small, Keyboard Common:Jumper_min_v2
- P1: footprint KiCad-SSD1306-0.91-OLED-4pin-128x32:SSD1306-0.91-OLED-4pin-128x32 -> Keyboard Common:SSD1306-0.91-OLED-4pin-128x32 doublesided
- moved P1 19.0 mm to (91.6, 56.4)
Connections:
- P1 pad 1: Net-(P1-Pin_1) -> GND
- P1 pad 2: Net-(P1-Pin_2) -> VCC
- P1 pad 3: Net-(P1-Pin_3) -> SCL
- P1 pad 4: Net-(P1-Pin_4) -> SDA
Routing:
- net unconnected-(P1-0-PadA): track 0.00 -> 3.08 mm
- net Net-(P1-Pin_4): track 3.08 -> 0.00 mm
- net unconnected-(P1-0-PadD): track 0.00 -> 3.02 mm
- net Net-(P1-Pin_1): track 3.02 -> 0.00 mm
- net unconnected-(P1-0-PadB): track 0.00 -> 3.02 mm
- net Net-(P1-Pin_3): track 3.02 -> 0.00 mm
- net unconnected-(P1-0-PadC): track 0.00 -> 2.95 mm
- net Net-(P1-Pin_2): track 2.95 -> 0.00 mm
- net GND: track 192.1 -> 194.7 mm
