File: Lotus 58 USB-C/v1.40/Lotus58_Glow_140.kicad_pcb (KiCad board)
At the start: 2 copper layers, 139.1 x 107.7 mm, 118 parts, among them J3 USB_C_Receptacle_USB2.0, P1 OLED, SW1 Kailh hotswap Choc V1 socket, SW10 Kailh hotswap Choc V1 socket, SW11 Kailh hotswap Choc V1 socket, SW12 Kailh hotswap Choc V1 socket, SW13 Kailh hotswap Choc V1 socket, SW14 Kailh hotswap Choc V1 socket, SW15 Kailh hotswap Choc V1 socket, SW16 Kailh hotswap Choc V1 socket, SW17 Kailh hotswap Choc V1 socket, SW18 Kailh hotswap Choc V1 socket, SW19 Kailh hotswap Choc V1 socket, SW2 Kailh hotswap Choc V1 socket, SW20 Kailh hotswap Choc V1 socket, SW21 Kailh hotswap Choc V1 socket, SW22 Kailh hotswap Choc V1 socket, SW23 Kailh hotswap Choc V1 socket, SW24 Kailh hotswap Choc V1 socket, SW25 Kailh hotswap Choc V1 socket, SW26 Kailh hotswap Choc V1 socket, SW27 Kailh hotswap Choc V1 socket, SW28 Kailh hotswap Choc V1 socket, SW29 Kailh hotswap Choc V1 socket, SW3 Kailh hotswap Choc V1 socket, SW30 Rotary_Encoder_Switch, SW32 MSK12C02, SW33 MSK12C02, SW4 Kailh hotswap Choc V1 socket, SW5 Kailh hotswap Choc V1 socket, SW6 Kailh hotswap Choc V1 socket, SW7 Kailh hotswap Choc V1 socket, SW8 Kailh hotswap Choc V1 socket, SW9 Kailh hotswap Choc V1 socket, U1 ProMicro, U2 SRV05-4

Commit message: Add voltage translator for LEDs with RP2040
* Added voltage translator
  - Routed USB Raw 5V from controller board to LED translator for use by
    LEDs
* Rerouted power link between boards to use USB Raw 5V instead of
  controller VCC
* Added additional backside placement for components
* Fixed schematic parity with pcb
Parts:
- added U3: SRV05-4, Package_TO_SOT_SMD:SOT-23-6, B.Cu at (91.8, 83.8)
- added U4: SN74LVC1T45DBVR, Spencer-Custom:DBV0006A_N, F.Cu at (114.0, 38.6)
- added U5: SN74LVC1T45DBVR, Spencer-Custom:DBV0006A_N, B.Cu at (114.0, 38.6)
- FB1: value Ferrite Beads -> Ferrite Bead
- moved SW32 14.6 mm to (123.4, 37.5)
- moved SW33 14.6 mm to (123.4, 37.5)
- moved RES1 12.7 mm to (106.2, 36.9)
- moved RES2 12.7 mm to (106.2, 36.9)
- moved Logo1 1.65 mm to (194.2, 43.0)
- moved Logo2 1.65 mm to (194.4, 43.0)
Connections:
- net /VCC_LINK renamed /5V_LINK
- FB1 pad 2: VCC -> +5V
- JP1 pad 2: VCC -> +5V
- JP2 pad 2: VCC -> +5V
- LED1 pad 4: LED -> LED_5V
- LED30 pad 4: LED -> LED_5V
- SW32 pad COM: VCC -> +5V
- SW33 pad COM: VCC -> +5V
- U1 pad 24: unconnected-(U1-RAW-Pad24) -> +5V
- U2 pad 5: VCC -> +5V
Routing:
- net +5V: track 0.00 -> 112.8 mm, vias 0 -> 6
- net LED_5V: track 0.00 -> 36.0 mm, vias 0 -> 4
- net LED: track 54.5 -> 31.8 mm
- net RESET: track 44.4 -> 31.9 mm
- net VCC: track 90.6 -> 83.8 mm, vias 6 -> 7
- net Net-(LED1-DOUT): track 25.5 -> 31.8 mm
- net /PWR_KEY: track 752.0 -> 745.6 mm, vias 44 -> 42
- net GND: track 165.6 -> 171.6 mm, vias 87 -> 90
- net DATA: track 66.7 -> 71.6 mm
- net /PWR_GLOW: track 319.4 -> 315.6 mm, vias 9 -> 10
- net SDA: track 44.3 -> 45.8 mm
- net /5V_LINK: track 9.66 -> 8.60 mm
- net SCL: track 35.9 -> 35.2 mm
Other:
- board text added: "Choc V1 Edition"
